File: project/machine that draw.kicad_sch (KiCad schematic)
At the start: 15 parts, among them J1 SD_Card_Device, J2 SSD1306 / 1 GND / 2 VCC / 3 S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, J3 limit switch, J4 limit switch, J5 Conn_01x04, J6 Conn_01x04, U1 ESP32-S3-UNO, U2 R-78E5.0-1.0

Commit message: schematics
Parts:
- removed C1: 100uF, symbol makerspace-unilasalle:C
- added C1: C_Polarized_Small, symbol Device:C_Polarized_Small
- added C4, C6, C8: 10uF, symbol makerspace-unilasalle:C
- added C5: 100uF, symbol Device:C_Polarized_Small
- added C7: 100nF, symbol makerspace-unilasalle:C
- added J7: Barrel_Jack, Connector_BarrelJack:BarrelJack_Horizontal, symbol Connector:Barrel_Jack
- added JP1, JP2, JP3, JP4, JP5, JP6: Jumper_2_Open, symbol Jumper:Jumper_2_Open
- A1: value Module-A4988 -> Driver_X
- A2: value Module-A4988 -> Driver_Y
- C2, C3: footprint (none) -> makerspace-unilasalle:C_1206
- J1: value SD_Card_Device -> SD_Card; footprint (none) -> makerspace-unilasalle:SD_Hirose_DM1AA_SF_PEJ82
- J2: footprint (none) -> Connector_PinHeader_2.54mm:PinHeader_1x04_P2.54mm_Vertical
- J3: value limit switch -> limit switch_X; footprint (none) -> Connector_PinHeader_2.54mm:PinHeader_1x03_P2.54mm_Vertical
- J4: value limit switch -> limit switch_Y; footprint (none) -> Connector_PinHeader_2.54mm:PinHeader_1x03_P2.54mm_Vertical
- J5: value Conn_01x04 -> Motor_X; footprint (none) -> Connector_PinHeader_2.54mm:PinHeader_1x04_P2.54mm_Vertical
- J6: value Conn_01x04 -> motor_Y; footprint (none) -> Connector_PinHeader_2.54mm:PinHeader_1x04_P2.54mm_Vertical
- R1, R2: value 10k -> 4.7K; footprint (none) -> makerspace-unilasalle:R_1206
- U1: footprint PCM_Espressif:ESP32-S3-DevKitC -> makerspace-unilasalle:ESP_S3_UNO
- U2: value R-78E5.0-1.0 -> Regulateur; footprint Converter_DCDC:Converter_DCDC_RECOM_R-78E-0.5_THT -> makerspace-unilasalle:Converter_DCDC_RECOM_R-78E-0.5_THT
Connections:
- net +12V: now also C3.1, U2.1 (IN), C1.1, C5.1, J7.1
- net +3V3: now also J2.2 (Pin_2), R1.1, R2.1, C7.2, C8.2; no longer C2.2, U2.3 (OUT)
- net +5V: now also C2.2, U1.8 (VIN), U2.3 (OUT), C4.1, C6.1; no longer C3.1, J2.2 (Pin_2), J3.1 (Pin_1), J4.1 (Pin_1), R1.1, R2.1, U1.2 (5V), U2.1 (IN)
- net GND: now also C1.2, C5.2, C7.1, C8.1, J7.2, JP1.1 (A), JP2.1 (A), JP3.1 (A), JP4.1 (A), JP5.1 (A), JP6.1 (A)
- net ENA: now reaches U1.24 (GPIO46)
- net ENA: now also A1.9 (~{ENABLE}), A2.9 (~{ENABLE})
- net STEP_Y: now reaches U1.25 (GPIO10/ADC1_CH9)
- net STEP_Y: now also A2.15 (STEP)
- net DIR_Y: now reaches U1.26 (GPIO11/ADC2_CH0)
- net DIR_Y: now also A2.16 (DIR)
- removed net GPIO 1: A1.10 (MS1), A2.10 (MS1), U1.10 (GPIO1/ADC1_CH0)
- removed net GPIO 12: A1.15 (STEP), A2.15 (STEP), U1.28 (GPIO12/ADC2_CH1)
- removed net GPIO 13: A1.16 (DIR), A2.16 (DIR), U1.27 (GPIO13/ADC2_CH2)
- removed net GPIO 14: A1.9 (~{ENABLE}), A2.9 (~{ENABLE}), U1.22 (GPIO14/ADC2_CH3)
- removed net GPIO 2: A1.11 (MS2), A2.11 (MS2), U1.9 (GPIO2/ADC1_CH1)
- removed net GPIO 3: A1.12 (MS3), A2.12 (MS3), U1.21 (GPIO3/ADC1_CH2)
- new net: A1.12 (MS3), JP6.2 (B)
- new net: A2.10 (MS1), JP1.2 (B)
- new net: C4.2, J4.1 (Pin_1)
- new net: A1.11 (MS2), JP5.2 (B)
- new net: A2.11 (MS2), JP2.2 (B)
- new net: A2.12 (MS3), JP3.2 (B)
- new net: A1.10 (MS1), JP4.2 (B)
- new net: C6.2, J3.1 (Pin_1)
- new net DIR_X: A1.16 (DIR), U1.28 (GPIO12/ADC2_CH1)
- new net LIMIT_X: J3.3 (Pin_3), U1.10 (GPIO1/ADC1_CH0)
- new net LIMIT_Y: J4.3 (Pin_3), U1.9 (GPIO2/ADC1_CH1)
- new net STEP_X: A1.15 (STEP), U1.27 (GPIO13/ADC2_CH2)
- now unconnected: U1.20 (GPIO20/USB_D+)
- no-connect marks 0 -> 15
Other:
- moved on the sheet: A1, A2, J2, J3, J5, J6

Commit message: Created PCB file
Parts:
- removed JP1, JP2, JP3, JP4, JP5, JP6: Jumper_2_Open, symbol Jumper:Jumper_2_Open
- added J8, J9: Conn_02x03_Odd_Even, Connector_PinHeader_2.54mm:PinHeader_2x03_P2.54mm_Vertical, symbol Connector_Generic:Conn_02x03_Odd_Even
- C1, C5: footprint (none) -> Capacitor_THT:CP_Radial_D8.0mm_P3.50mm
- C4, C6, C7, C8: footprint (none) -> makerspace-unilasalle:C_1206
Connections:
- net GND: now also J8.1 (Pin_1), J8.3 (Pin_3), J8.5 (Pin_5), J9.1 (Pin_1), J9.3 (Pin_3), J9.5 (Pin_5)
- net at A1.12 (MS3): now also J9.6 (Pin_6)
- net at A2.10 (MS1): now also J8.2 (Pin_2)
- net at A1.11 (MS2): now also J9.4 (Pin_4)
- net at A2.11 (MS2): now also J8.4 (Pin_4)
- net at A2.12 (MS3): now also J8.6 (Pin_6)
- net at A1.10 (MS1): now also J9.2 (Pin_2)

Commit message: finalisation pcb
Parts:
- removed C8: 10uF, makerspace-unilasalle:C_1206, symbol makerspace-unilasalle:C
- added C9: 10 uF, Capacitor_SMD:C_1206_3216Metric_Pad1.33x1.80mm_HandSolder, symbol makerspace-unilasalle:C
- C4: footprint makerspace-unilasalle:C_1206 -> Capacitor_SMD:C_1206_3216Metric_Pad1.33x1.80mm_HandSolder
- C7: value 100nF -> 10 uF; footprint makerspace-unilasalle:C_1206 -> Capacitor_SMD:C_1206_3216Metric_Pad1.33x1.80mm_HandSolder
Connections:
- net +5V: now also J3.1 (Pin_1), J4.1 (Pin_1), C9.2
- net DIR_Y: now also U1.25 (GPIO10/ADC1_CH9); no longer U1.26 (GPIO11/ADC2_CH0)
- net GND: now also C4.2, C6.2, C9.1
- net STEP_Y: now also U1.26 (GPIO11/ADC2_CH0); no longer U1.25 (GPIO10/ADC1_CH9)
- net at J8.2 (Pin_2): now also A2.12 (MS3); no longer A2.10 (MS1)
- net at J8.6 (Pin_6): now also A2.10 (MS1); no longer A2.12 (MS3)
- net at J9.2 (Pin_2): now also A1.12 (MS3); no longer A1.10 (MS1)
- net at J9.6 (Pin_6): now also A1.10 (MS1); no longer A1.12 (MS3)
Other:
- moved on the sheet: C6, J2, R2

Commit message: fix wiring problems
Connections:
- net +12V: now also U1.8 (VIN)
- net +5V: no longer U1.8 (VIN)
